File: KiCad Files/MicroDev128.kicad_pcb (KiCad board)
At the start: 4 copper layers, 49.1 x 17.8 mm, 32 parts, among them J1 UPDI, J3 GPIO, J4 PWR and ANALOG, SW1 SW_SP3T, SW2 RST, U1 AVR128DB32x-xRXB, U2 LT8653SEV_PBF

Commit message: Updated For Production
Parts:
- moved G*** 101.9 mm to (179.3, 120.1)
Changed lines of the file:
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@@
 	(footprint "LOGO"
 		(layer "B.Cu")
-		(at 95.5 62.1 180)
+		(at 179.270431 120.117018 180)
 		(property "Reference" "G***"
 			(at 0 0 0)
@@
 	)
 	(zone
-		(net "GND")
-		(layer "F.Cu")
-		(name "Top GND")
-		(hatch edge 0.5)
-		(priority 1)
-		(connect_pads
-			(clearance 0.208)
-		)
-		(min_thickness 0.25)
-		(fill yes
-			(thermal_gap 0.5)
-			(thermal_bridge_width 0.5)
-			(island_removal_mode 2)
-			(island_area_min 10)
-		)
-		(polygon
-			(pts
-				(xy 156.723083 110.63) (xy 156.783083 128.45) (xy 205.703083 128.28) (xy 205.713083 110.66)
-			)
-		)
-	)
-	(zone
 		(net "Net-(D3-K)")
 		(layer "F.Cu")
@@
 			)
 		)
+	)
+	(zone
+		(net "GND")
+		(layer "F.Cu")
+		(name "Top GND")
+		(hatch edge 0.5)
+		(priority 1)
+		(connect_pads
+			(clearance 0.208)
+		)
+		(min_thickness 0.25)
+		(fill yes
+			(thermal_gap 0.5)
+			(thermal_bridge_width 0.5)
+			(island_removal_mode 2)
+			(island_area_min 10)
+		)
+		(polygon
+			(pts
+				(xy 156.723083 110.63) (xy 156.783083 128.45) (xy 205.703083 128.28) (xy 205.713083 110.66)
+			)
+		)
